File: schematics/MotorDriver2/MotorDriver.kicad_pcb (KiCad board)
At the start: 2 copper layers, 37 parts, among them J1 9Vin, J10 MotorB, J2 ICSP, J3 FTDI, J4 I2C, J5 3v3out, J6 AnalogPins, J7 WheelEncA, J8 WheelEncB, J9 MotorA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

Commit message: Dis
Parts:
- C11, C2, C3, C4, C6, C7, C8: footprint Capacitor_SMD:C_1206_3216Metric -> Capacitor_SMD:C_0402_1005Metric
- D1, D2: footprint Diode_SMD:D_1206_3216Metric -> Diode_SMD:D_0402_1005Metric
- R1, R2, R3, R4, R5: footprint Resistor_SMD:R_1206_3216Metric -> Resistor_SMD:R_0402_1005Metric
- Y1: value HC-49SM16MHz20pF30ppm -> 16MHz; footprint Crystal:Crystal_SMD_0603-2Pin_6.0x3.5mm_HandSoldering -> Crystal:Crystal_SMD_HC49-SD
- moved H2 115.0 mm to (69.1, 149.4)
- moved H1 83.2 mm to (69.2, 106.2)
- moved H3 56.4 mm to (125.4, 149.1)
- moved H4 38.7 mm to (125.4, 105.9)
- moved J3 34.9 mm to (112.1, 110.2)
- moved D1 34.2 mm to (105.5, 141.7)
- moved R3 34.1 mm to (107.1, 142.9), turned to 270 degrees
- moved J1 33.4 mm to (85.9, 144.5), turned to 180 degrees
- moved C6 29.4 mm to (105.5, 144.2), turned to 0 degrees
- moved U2 29.2 mm to (97.5, 144.1)
- moved C5 28.9 mm to (102.0, 143.5)
- moved C1 25.6 mm to (93.0, 143.5)
- moved J5 24.6 mm to (111.4, 143.0), turned to 0 degrees
- moved Y1 23.0 mm to (97.2, 116.7), turned to 0 degrees
- moved C9 18.8 mm to (92.3, 123.1), turned to 90 degrees
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Connections:
- J9 pad 1: MOTORA1 -> MOTORA2
- J9 pad 2: MOTORA2 -> MOTORA1
Routing:
- net +3V3: track 145.0 -> 289.1 mm, vias 0 -> 7
- net GND: track 0.00 -> 57.6 mm, vias 0 -> 4
- net D3: track 0.00 -> 33.3 mm, vias 0 -> 1
- net MOTORA2: track 0.00 -> 31.5 mm
- net D2: track 0.00 -> 30.4 mm, vias 0 -> 1
- net +9V: track 17.4 -> 47.0 mm, vias 0 -> 2
- net MOTORA1: track 0.00 -> 25.9 mm
- net MOTORB2: track 0.00 -> 25.4 mm
- net MOTORB1: track 0.00 -> 21.8 mm
- net D4: track 0.00 -> 17.2 mm, vias 0 -> 2
- net D6: track 0.00 -> 13.6 mm, vias 0 -> 2
- net D10: track 0.00 -> 12.8 mm, vias 0 -> 2
- net D7: track 0.00 -> 11.5 mm, vias 0 -> 2
- net D8: track 0.00 -> 11.5 mm
- net D9: track 0.00 -> 11.0 mm, vias 0 -> 2
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- added copper zone on F.Cu, net GND
