File: schematics/RobotHat/RobotHat.sch (KiCad schematic (older format))
At the start: 53 parts, among them J1 9Vin, J10 MotorA, J11 MotorB, J12 Raspberry_Pi_2_3, J2 5Vout, J4 ATMega_ICSP, J5 ATMega_FTDI, J6 I2C, J7 ATMega AnalogPins, J8 WheelEncA, J9 WheelEncB, Q1 AO3401A, Q2 2N7002, Q3 2N7002, SW1 Reset, U1 ATmega328P-AU, U2 LM2596S-5, U3 TB6612FNG, Y1 16MHz

Commit message: Hehe
Parts:
- removed C2, C4: 15pF, Capacitor_SMD:C_0402_1005Metric, symbol Device:C
- removed Y1: 16MHz, Crystal:Crystal_HC49-4H_Vertical, symbol Device:Crystal
- added Y1: 16Mhz, RobotHat:CSTCE16M0V53-R0, symbol Device:Crystal_GND3
- L1: footprint Inductor_THT:L_Radial_D8.7mm_P5.00mm_Fastron_07HCP -> RobotHat:YPRH1207-330M; Part No (none) -> C339951
- R10, R7, R8, R9: value 4.7k -> 10k
Connections:
- net GND: now also Y1.3
- net XTAL1: now also Y1.1
- net XTAL2: now also Y1.2
Other:
- moved on the sheet: Q2, Q3, R10, R7, R8, R9
Changed lines of the file:
@@
-$EndComp
-$Comp
-L Device:Crystal Y1
-U 1 1 617B9139
-P 4050 2900
-F 0 "Y1" H 3850 2800 50  0000 L CNN
-F 1 "16MHz" H 3200 2700 50  0000 L CNN
-F 2 "Crystal:Crystal_HC49-4H_Vertical" H 4050 2900 50  0001 C CNN
-F 3 "~" H 4050 2900 50  0001 C CNN
-	1    4050 2900
-	-1   0    0    1
-$EndComp
-$Comp
-L Device:C C4
-U 1 1 617FEF79
-P 4300 3150
-F 0 "C4" H 4185 3104 50  0000 R CNN
-F 1 "15pF" H 4185 3195 50  0000 R CNN
-F 2 "Capacitor_SMD:C_0402_1005Metric" H 4338 3000 50  0001 C CNN
-F 3 "~" H 4300 3150 50  0001 C CNN
-	1    4300 3150
-	-1   0    0    1
-$EndComp
-$Comp
-L Device:C C2
-U 1 1 618015EB
-P 3800 3150
-F 0 "C2" H 3685 3104 50  0000 R CNN
-F 1 "15pF" H 3685 3195 50  0000 R CNN
-F 2 "Capacitor_SMD:C_0402_1005Metric" H 3838 3000 50  0001 C CNN
-F 3 "~" H 3800 3150 50  0001 C CNN
-	1    3800 3150
-	-1   0    0    1
 $EndComp
 $Comp
@@
 XTAL2
 Wire Wire Line
-	3800 3300 4050 3300
-Wire Wire Line
-	4050 3400 4050 3300
-Connection ~ 4050 3300
-Wire Wire Line
-	4050 3300 4300 3300
-Wire Wire Line
-	3800 3000 3800 2900
-Wire Wire Line
 	3800 2900 3900 2900
 Wire Wire Line
-	4200 2900 4300 2900
-Wire Wire Line
-	4300 2900 4300 3000
-Wire Wire Line
 	3800 2900 3800 2550
 Wire Wire Line
 	3800 2550 4400 2550
-Connection ~ 3800 2900
-Wire Wire Line
-	4300 2900 4400 2900
-Connection ~ 4300 2900
 Text GLabel 4400 2550 2    50   Input ~ 0
 XTAL1
@@
 L power:+3.3V #PWR011
 U 1 1 61981A00
-P 8450 4200
-F 0 "#PWR011" H 8450 4050 50  0001 C CNN
-F 1 "+3.3V" H 8465 4373 50  0000 C CNN
-F 2 "" H 8450 4200 50  0001 C CNN
-F 3 "" H 8450 4200 50  0001 C CNN
-	1    8450 4200
+P 7400 4250
+F 0 "#PWR011" H 7400 4100 50  0001 C CNN
+F 1 "+3.3V" H 7415 4423 50  0000 C CNN
+F 2 "" H 7400 4250 50  0001 C CNN
+F 3 "" H 7400 4250 50  0001 C CNN
+	1    7400 4250
 	1    0    0    -1
 $EndComp
@@
 F 0 "L1" V 4500 1400 50  0000 C CNN
 F 1 "33uH" V 4700 1400 50  0000 C CNN
-F 2 "Inductor_THT:L_Radial_D8.7mm_P5.00mm_Fastron_07HCP" H 4600 1400 50  0001 C CNN
+F 2 "RobotHat:YPRH1207-330M" H 4600 1400 50  0001 C CNN
 F 3 "~" H 4600 1400 50  0001 C CNN
+F 4 "C339951" V 4600 1400 50  0001 C CNN "Part No"
 	1    4600 1400
 	0    1    1    0
@@
 Wire Wire Line
 	6150 3000 6150 3150
-Text GLabel 7800 4650 0    50   Input ~ 0
+Text GLabel 8150 4700 2    50   Input ~ 0
 SDA
-Text GLabel 8600 4650 2    50   Input ~ 0
+Text GLabel 7150 4700 0    50   Input ~ 0
 3v3_SDA
 $Comp
 L power:+5V #PWR040
 U 1 1 618E2D51
-P 8050 4200
-F 0 "#PWR040" H 8050 4050 50  0001 C CNN
-F 1 "+5V" H 8065 4373 50  0000 C CNN
-F 2 "" H 8050 4200 50  0001 C CNN
-F 3 "" H 8050 4200 50  0001 C CNN
-	1    8050 4200
+P 7800 4250
+F 0 "#PWR040" H 7800 4100 50  0001 C CNN
+F 1 "+5V" H 7815 4423 50  0000 C CNN
+F 2 "" H 7800 4250 50  0001 C CNN
+F 3 "" H 7800 4250 50  0001 C CNN
+	1    7800 4250
 	1    0    0    -1
 $EndComp
@@
 L Device:R R9
 U 1 1 618E7DE9
-P 8450 4400
-F 0 "R9" H 8520 4446 50  0000 L CNN
-F 1 "4.7k" H 8520 4355 50  0000 L CNN
-F 2 "Resistor_SMD:R_0402_1005Metric" V 8380 4400 50  0001 C CNN
-F 3 "~" H 8450 4400 50  0001 C CNN
-	1    8450 4400
+P 7400 4450
+F 0 "R9" H 7200 4500 50  0000 L CNN
+F 1 "10k" H 7200 4400 50  0000 L CNN
+F 2 "Resistor_SMD:R_0402_1005Metric" V 7330 4450 50  0001 C CNN
+F 3 "~" H 7400 4450 50  0001 C CNN
+	1    7400 4450
 	1    0    0    -1
 $EndComp
@@
 L Device:R R7
 U 1 1 618EF6E6
-P 8050 4400
-F 0 "R7" H 7850 4450 50  0000 L CNN
-F 1 "4.7k" H 7800 4350 50  0000 L CNN
-F 2 "Resistor_SMD:R_0402_1005Metric" V 7980 4400 50  0001 C CNN
-F 3 "~" H 8050 4400 50  0001 C CNN
-	1    8050 4400
-	1    0    0    -1
-$EndComp
-Wire Wire Line
-	8450 4200 8450 4250
-Wire Wire Line
-	8050 4200 8050 4250
-Wire Wire Line
-	8050 4550 8050 4650
-Wire Wire Line
-	8050 4650 7800 4650
-Wire Wire Line
-	8450 4650 8450 4550
-Wire Wire Line
-	8450 4650 8600 4650
-Wire Wire Line
-	8250 4350 8250 4250
-Wire Wire Line
-	8250 4250 8450 4250
-Connection ~ 8450 4250
+P 7800 4450
+F 0 "R7" H 7900 4500 50  0000 L CNN
+F 1 "10k" H 7900 4400 50  0000 L CNN
+F 2 "Resistor_SMD:R_0402_1005Metric" V 7730 4450 50  0001 C CNN
+F 3 "~" H 7800 4450 50  0001 C CNN
+	1    7800 4450
+	1    0    0    -1
+$EndComp
 $Comp
 L Device:R R8
 U 1 1 6195FCAA
-P 8100 5600
-F 0 "R8" H 7900 5650 50  0000 L CNN
-F 1 "4.7k" H 7850 5550 50  0000 L CNN
-F 2 "Resistor_SMD:R_0402_1005Metric" V 8030 5600 50  0001 C CNN
-F 3 "~" H 8100 5600 50  0001 C CNN
-	1    8100 5600
+P 7800 5500
+F 0 "R8" H 7850 5550 50  0000 L CNN
+F 1 "10k" H 7850 5450 50  0000 L CNN
+F 2 "Resistor_SMD:R_0402_1005Metric" V 7730 5500 50  0001 C CNN
+F 3 "~" H 7800 5500 50  0001 C CNN
+	1    7800 5500
 	1    0    0    -1
 $EndComp
@@
 L Device:R R10
 U 1 1 6196077A
-P 8500 5600
-F 0 "R10" H 8570 5646 50  0000 L CNN
-F 1 "4.7k" H 8570 5555 50  0000 L CNN
-F 2 "Resistor_SMD:R_0402_1005Metric" V 8430 5600 50  0001 C CNN
-F 3 "~" H 8500 5600 50  0001 C CNN
-	1    8500 5600
+P 7400 5500
+F 0 "R10" H 7200 5550 50  0000 L CNN
+F 1 "10k" H 7200 5450 50  0000 L CNN
+F 2 "Resistor_SMD:R_0402_1005Metric" V 7330 5500 50  0001 C CNN
+F 3 "~" H 7400 5500 50  0001 C CNN
+	1    7400 5500
 	1    0    0    -1
 $EndComp
@@
 L power:+5V #PWR044
 U 1 1 6196B419
-P 8100 5350
-F 0 "#PWR044" H 8100 5200 50  0001 C CNN
-F 1 "+5V" H 8115 5523 50  0000 C CNN
-F 2 "" H 8100 5350 50  0001 C CNN
-F 3 "" H 8100 5350 50  0001 C CNN
-	1    8100 5350
+P 7800 5250
+F 0 "#PWR044" H 7800 5100 50  0001 C CNN
+F 1 "+5V" H 7815 5423 50  0000 C CNN
+F 2 "" H 7800 5250 50  0001 C CNN
+F 3 "" H 7800 5250 50  0001 C CNN
+	1    7800 5250
 	1    0    0    -1
 $EndComp
@@
 L power:+3.3V #PWR045
 U 1 1 6196BBEA
-P 8500 5350
-F 0 "#PWR045" H 8500 5200 50  0001 C CNN
-F 1 "+3.3V" H 8515 5523 50  0000 C CNN
-F 2 "" H 8500 5350 50  0001 C CNN
-F 3 "" H 8500 5350 50  0001 C CNN
-	1    8500 5350
-	1    0    0    -1
-$EndComp
-Text GLabel 7800 5900 0    50   Input ~ 0
+P 7400 5250
+F 0 "#PWR045" H 7400 5100 50  0001 C CNN
+F 1 "+3.3V" H 7415 5423 50  0000 C CNN
+F 2 "" H 7400 5250 50  0001 C CNN
+F 3 "" H 7400 5250 50  0001 C CNN
+	1    7400 5250
+	1    0    0    -1
+$EndComp
+Text GLabel 8150 5800 2    50   Input ~ 0
 SCL
-Text GLabel 8650 5900 2    50   Input ~ 0
+Text GLabel 7200 5800 0    50   Input ~ 0
 3v3_SCL
 Wire Wire Line
-	8100 5450 8100 5350
-Wire Wire Line
-	8500 5450 8500 5400
-Wire Wire Line
-	8300 5600 8300 5400
-Wire Wire Line
-	8300 5400 8500 5400
-Connection ~ 8500 5400
-Wire Wire Line
-	8500 5400 8500 5350
-Wire Wire Line
-	8500 5750 8500 5900
-Wire Wire Line
-	8500 5900 8650 5900
-Wire Wire Line
-	8100 5750 8100 5900
-Wire Wire Line
-	8100 5900 7800 5900
+	7400 5350 7400 5250
+Wire Wire Line
+	7800 5650 7800 5800
+Wire Wire Line
+	7400 5650 7400 5800
+Wire Wire Line
+	7400 5800 7200 5800
 $Comp
 L power:+5V #PWR0106
@@
 L Transistor_FET:2N7002 Q2
 U 1 1 61818AAA
-P 8250 4550
-F 0 "Q2" V 8499 4550 50  0000 C CNN
-F 1 "2N7002" V 8590 4550 50  0000 C CNN
-F 2 "Package_TO_SOT_SMD:SOT-23" H 8450 4475 50  0001 L CIN
-F 3 "https://www.onsemi.com/pub/Collateral/NDS7002A-D.PDF" H 8250 4550 50  0001 L CNN
-	1    8250 4550
-	0    -1   1    0
-$EndComp
-Connection ~ 8450 4650
-Connection ~ 8050 4650
+P 7600 4600
+F 0 "Q2" V 7849 4600 50  0000 C CNN
+F 1 "2N7002" V 7940 4600 50  0000 C CNN
+F 2 "Package_TO_SOT_SMD:SOT-23" H 7800 4525 50  0001 L CIN
+F 3 "https://www.onsemi.com/pub/Collateral/NDS7002A-D.PDF" H 7600 4600 50  0001 L CNN
+	1    7600 4600
+	0    1    1    0
+$EndComp
 $Comp
 L Transistor_FET:2N7002 Q3
 U 1 1 618386BA
-P 8300 5800
-F 0 "Q3" V 8549 5800 50  0000 C CNN
-F 1 "2N7002" V 8640 5800 50  0000 C CNN
-F 2 "Package_TO_SOT_SMD:SOT-23" H 8500 5725 50  0001 L CIN
-F 3 "https://www.onsemi.com/pub/Collateral/NDS7002A-D.PDF" H 8300 5800 50  0001 L CNN
-	1    8300 5800
-	0    -1   1    0
-$EndComp
-Connection ~ 8500 5900
-Connection ~ 8100 5900
+P 7600 5700
+F 0 "Q3" V 7849 5700 50  0000 C CNN
+F 1 "2N7002" V 7940 5700 50  0000 C CNN
+F 2 "Package_TO_SOT_SMD:SOT-23" H 7800 5625 50  0001 L CIN
+F 3 "https://www.onsemi.com/pub/Collateral/NDS7002A-D.PDF" H 7600 5700 50  0001 L CNN
+	1    7600 5700
+	0    1    1    0
+$EndComp
+Connection ~ 7800 5800
+Connection ~ 7400 5800
+Wire Wire Line
+	7800 5250 7800 5350
+Wire Wire Line
+	7400 4250 7400 4300
+Wire Wire Line
+	7400 4600 7400 4700
+Wire Wire Line
+	7400 4700 7150 4700
+Connection ~ 7400 4700
+Wire Wire Line
+	7800 4700 8150 4700
+Wire Wire Line
+	7800 4700 7800 4600
+Connection ~ 7800 4700
+Wire Wire Line
+	7800 4300 7800 4250
+Wire Wire Line
+	7800 5800 8150 5800
+Wire Wire Line
+	7600 4400 7600 4300
+Wire Wire Line
+	7600 4300 7400 4300
+Connection ~ 7400 4300
+Wire Wire Line
+	7600 5500 7600 5350
+Wire Wire Line
+	7600 5350 7400 5350
+Connection ~ 7400 5350
+$Comp
+L Device:Crystal_GND3 Y1
+U 1 1 61934016
+P 4050 2900
+F 0 "Y1" H 4050 3168 50  0000 C CNN
+F 1 "16Mhz" H 4050 3077 50  0000 C CNN
+F 2 "RobotHat:CSTCE16M0V53-R0" H 4050 2900 50  0001 C CNN
+F 3 "~" H 4050 2900 50  0001 C CNN
+	1    4050 2900
+	1    0    0    -1
+$EndComp
+Wire Wire Line
+	4200 2900 4400 2900
+Wire Wire Line
+	4050 3100 4050 3400
 $EndSCHEMATC
