File: schematics/RobotHat/RobotHat.sch (KiCad schematic (older format))
At the start: 49 parts, among them J1 9Vin, J10 MotorA, J11 MotorB, J12 Raspberry_Pi_2_3, J2 5Vout, J4 ATMega_ICSP, J5 ATMega_FTDI, J6 I2C, J7 ATMega AnalogPins, J8 WheelEncA, J9 WheelEncB, Q1 AO3401A, Q2 2N7002, Q3 2N7002, SW1 Reset, U1 ATmega328P-AU, U2 LM2596S-5, U3 TB6612FNG, Y1 16Mhz

Commit message: It
Parts:
- removed R1, R2: 10k, Resistor_SMD:R_1206_3216Metric, symbol Device:R
- removed Y1: 16Mhz, RobotHat:CSTCE16M0V53-R0, symbol Device:Crystal_GND3
- added C2, C4: 22pF, Diode_SMD:D_0603_1608Metric, symbol Device:C
- added J12: TFT_SPI_DISPLAY, Connector_PinHeader_2.54mm:PinHeader_2x05_P2.54mm_Vertical, symbol Connector_Generic:Conn_01x09
- added Y1: Crystal, Crystal:Crystal_HC49-4H_Vertical, symbol Device:Crystal
- C1: Part (none) -> C127971; Part # C127971 -> (none)
- C10: Field4 C24497 -> (none)
- C11, C7: Part (none) -> C307331; Part # C24497 -> (none)
- C3, C6: footprint Capacitor_SMD:C_0402_1005Metric -> Capacitor_SMD:C_1206_3216Metric; Part (none) -> C307331; Part # C307331 -> (none)
- C5: Part (none) -> C371974; Part # C371974 -> (none)
- C8: Part (none) -> C134721; Part # C134721 -> (none)
- C9: Part # C24497 -> (none)
- D1: Part (none) -> C8678; Part # C8678 -> (none)
- D2, D4: value GREEN -> RED; footprint Diode_SMD:D_0402_1005Metric -> Diode_SMD:D_0603_1608Metric; Part (none) -> C2286
- D3: footprint Diode_SMD:D_0402_1005Metric -> Diode_SMD:D_0603_1608Metric; Part (none) -> C2286; Part # C130719 -> (none)
- L1: Part (none) -> C339951; Part # C339951 -> (none)
- Q1: JLCPCB Part # C15127 -> (none); Part (none) -> C15127
- Q2, Q3: Part (none) -> C8545; Part # C8545 -> (none)
- R1: renamed from R3; footprint Resistor_SMD:R_0805_2012Metric -> Resistor_SMD:R_0603_1608Metric; Part (none) -> C25804; Part # C17724 -> (none)
- R2: renamed from R4; footprint Resistor_SMD:R_0402_1005Metric -> Resistor_SMD:R_0603_1608Metric; Part (none) -> C23138; Part # C25741 -> (none)
- R3: renamed from R5; footprint Resistor_SMD:R_0402_1005Metric -> Resistor_SMD:R_0603_1608Metric; Part (none) -> C23138; Part # C25741 -> (none)
- R4: renamed from R6; footprint Resistor_SMD:R_0402_1005Metric -> Resistor_SMD:R_0603_1608Metric; Part (none) -> C23138; Part # C25741 -> (none)
- R5: renamed from R9; footprint Resistor_SMD:R_0805_2012Metric -> Resistor_SMD:R_0603_1608Metric; Part (none) -> C25804; Part # C17724 -> (none)
- R6: renamed from R10; footprint Resistor_SMD:R_0805_2012Metric -> Resistor_SMD:R_0603_1608Metric; Part (none) -> C25804; Part # C17724 -> (none)
- R7: footprint Resistor_SMD:R_0805_2012Metric -> Resistor_SMD:R_0603_1608Metric; Part (none) -> C25804
- R8: footprint Resistor_SMD:R_0805_2012Metric -> Resistor_SMD:R_0603_1608Metric; Part (none) -> C25804; Part # C17724 -> (none)
- SW1: footprint Button_Switch_SMD:SW_Push_1P1T_NO_Vertical_Wuerth_434133025816 -> MyFootprints:TS-1187A-B-A-B_PushButton; Part (none) -> C318884
- U1: Part (none) -> C14877; Part # C14877 -> (none)
- U2: Part (none) -> C194349; Part # C194349 -> (none)
- U3: Part (none) -> C141517; Part # C141517 -> (none)
- renumbered J7 to J10, J12 to J11, J4 to J3, J5 to J4, J6 to J5, J8 to J6, J9 to J7, J10 to J8, J11 to J9
Connections:
- net +3V3: now also J12.1 (Pin_1)
- net GND: now also C2.2, C4.2, J12.2 (Pin_2)
- net XTAL1: now also C2.1, Y1.1
- net XTAL2: now also C4.1, Y1.2
- net TFT_LED: now reaches J11.12 (GPIO18/PWM0)
- net TFT_LED: now also J12.8 (Pin_8)
- net TFT_DCRS: now reaches J11.18 (GPIO24)
- net TFT_DCRS: now also J12.5 (Pin_5)
- net TFT_RESET: now reaches J11.22 (GPIO25)
- net TFT_RESET: now also J12.4 (Pin_4)
- net TFT_CS: now reaches J11.24 (~CE0~/GPIO8)
- net TFT_CS: now also J12.3 (Pin_3)
- net RPI_MOSI: now reaches J11.35 (GPIO19/MISO1)
- net RPI_MOSI: now also J12.6 (Pin_6)
- net RPI_MISO: now reaches J11.38 (GPIO20/MOSI1)
- net RPI_MISO: now also J12.9 (Pin_9)
- net RPI_SCLK: now reaches J11.40 (GPIO21/SCLK1)
- net RPI_SCLK: now also J12.7 (Pin_7)
- no-connect marks 26 -> 19
