File: schematics/RobotHatPerf/RobotHat.sch (KiCad schematic (older format))
At the start: 49 parts, among them J1 9Vin, J10 MotorA, J11 MotorB, J12 Raspberry_Pi_2_3, J2 5Vout, J4 ATMega_ICSP, J5 ATMega_FTDI, J6 I2C, J7 ATMega AnalogPins, J8 WheelEncA, J9 WheelEncB, Q1 AO3401A, Q2 2N7002, Q3 2N7002, SW1 Reset, U1 ATmega328P-AU, U2 LM2596S-5, U3 TB6612FNG, Y1 16Mhz

Commit message: other
Parts:
- removed C10, C11, C9: 100nF, Capacitor_SMD:C_1206_3216Metric, symbol Device:C
- removed C8: 10uf, Capacitor_SMD:CP_Elec_4x5.3, symbol Device:CP
- removed J7: ATMega AnalogPins, Connector_PinSocket_2.54mm:PinSocket_2x03_P2.54mm_Horizontal, symbol Connector_Generic:Conn_02x03_Odd_Even
- removed R1, R2: 10k, Resistor_SMD:R_1206_3216Metric, symbol Device:R
- removed U1: ATmega328P-AU, Package_QFP:TQFP-32_7x7mm_P0.8mm, symbol MCU_Microchip_ATmega:ATmega328P-AU
- removed U3: TB6612FNG, Package_SO:SSOP-24_5.3x8.2mm_P0.65mm, symbol Driver_Motor:TB6612FNG
- removed Y1: 16Mhz, RobotHat:CSTCE16M0V53-R0, symbol Device:Crystal_GND3
- added C2, C3: 22pF, Capacitor_SMD:C_1206_3216Metric, symbol Device:C
- added C8: 100nF, Capacitor_SMD:C_1206_3216Metric, symbol Device:C
- added J8: ATMega AnalogPins, Connector_PinSocket_2.54mm:PinSocket_1x04_P2.54mm_Horizontal, symbol Connector_Generic:Conn_02x02_Odd_Even
- added U1: ATmega328P-PU, Package_DIP:DIP-28_W7.62mm, symbol MCU_Microchip_ATmega:ATmega328P-PU
- added U3: TB6612FNG_Breakout, MyFootprints:TB6612FNG_Breakout, symbol RobotHat:TB6612FNG_Breakout
- added Y1: 16MHz, Crystal:Crystal_HC49-U_Vertical, symbol Device:Crystal
- C1: Part (none) -> C127971; Part # C127971 -> (none)
- C4: renamed from C3; Part (none) -> C307331; Part # C307331 -> (none)
- C5: Part (none) -> C371974; Part # C371974 -> (none)
- C6: Part (none) -> C307331; Part # C307331 -> (none)
- C7: Part (none) -> C24497; Part # C24497 -> (none)
- D1: Part (none) -> C8678; Part # C8678 -> (none)
- D2, D4: Part (none) -> C130719
- D3: Part (none) -> C130719; Part # C130719 -> (none)
- L1: Part (none) -> C339951; Part # C339951 -> (none)
- Q1: JLCPCB Part # C15127 -> (none); Part (none) -> C15127
- Q2, Q3: Part (none) -> C8545; Part # C8545 -> (none)
- R1: renamed from R3; Part (none) -> C17724; Part # C17724 -> (none)
- R2: renamed from R4; Part (none) -> C25741; Part # C25741 -> (none)
- R3: renamed from R5; Part (none) -> C25741; Part # C25741 -> (none)
- R4: renamed from R6; Part (none) -> C25741; Part # C25741 -> (none)
- R5: renamed from R9; Part (none) -> C17724; Part # C17724 -> (none)
- R6: renamed from R10; Part (none) -> C17724; Part # C17724 -> (none)
- R7: Part (none) -> C17724
- R8: Part (none) -> C17724; Part # C17724 -> (none)
- SW1: footprint Button_Switch_SMD:SW_Push_1P1T_NO_Vertical_Wuerth_434133025816 -> MyFootprints:TS-1187A-B-A-B_PushButton; Part (none) -> C318884
- U2: Part (none) -> C194349; Part # C194349 -> (none)
- renumbered J11 to J10, J12 to J11, J4 to J3, J5 to J4, J6 to J5, J8 to J6, J9 to J7, J10 to J9
Connections:
- net labels removed: A6, A7
- wire segments 101 -> 87

Commit message: This
Parts:
- added BT? (x2): 18650, symbol Device:Battery_Cell
- added D? (x2): SS34, RobotHat:SS34, symbol Diode:1N5822
- added J?: Barrel_Jack, symbol Connector:Barrel_Jack
- added Q?: AO3401A, Package_TO_SOT_SMD:SOT-23, symbol Transistor_FET:AO3401A
- added R?: 10k, Resistor_SMD:R_0805_2012Metric, symbol Device:R
- added U?: TP5100_Carging_Module, symbol MySymbols:TP5100_Carging_Module
- added U?: BMS_18650_2S_Module, symbol MySymbols:BMS_18650_2S_Module
Connections:
- net +9V: now also D?.1 (K), D?.1 (K)
- net GND: now also J?.2, R?.2, U?.~ (P-), U?.~ (Vout)
- new net: D?.2 (A), J?.1, Q?.1 (G), R?.1, U?.~ (Vout)
- new net: Q?.2 (S), U?.~ (P-), U?.~ (Vout)
- new net: BT?.1 (+), U?.~ (P-)
- new net: BT?.1 (+), BT?.2 (-), U?.~ (P-)
- new net: BT?.2 (-), U?.~ (P-)
- new net: D?.2 (A), Q?.3 (D)
Other:
- note added: "Battery Charging/Discharging Circuite"
- note added: "This is to prevent backflow into battery when \nexternal plugged in\n"
